Commit message: Add arm_controllers pkg, franka urdf base linked to world eflin urdf clean

File: elfin_description/urdf/elfin3.urdf.xacro (robot description, xacro)
@@ -46,5 +46,6 @@
         rpy="0 0 0" />
       <geometry>
-        <mesh filename="package://elfin_description/meshes/elfin3/elfin_base.STL"/>
+        <mesh
+          filename="package://elfin_description/meshes/elfin3/elfin_base.STL" />
       </geometry>
       <material
@@ -56,5 +57,6 @@
         rpy="0 0 0" />
       <geometry>
-        <mesh filename="package://elfin_description/meshes/elfin3/elfin_base.STL" />
+        <mesh
+          filename="package://elfin_description/meshes/elfin3/elfin_base.STL" />
       </geometry>
     </collision>

File: franka_description/urdf/fp3_franka_hand.urdf (robot description, URDF)
Before this commit: robot fp3, 14 links, 13 joints
Links:
- added link world
Joints:
- added joint world_base: type fixed, parent world, child base, origin xyz=0 0 0 rpy=0 0 0
